Commit message: Update lolo and sam robot_description and meshes

File: lolo_stonefish_sim/data/lolo_auv/lolo_auv.urdf.xacro (robot description, xacro)
@@ -1,8 +1,11 @@
 <?xml version="1.0"?>
 <robot name="lolo_auv" xmlns:xacro="http://www.ros.org/wiki/xacro">
-  <xacro:property name="visual_mesh_file" value="file://$(find lolo_stonefish_sim)/data/lolo_auv/mesh/lolo.obj"/>
-  <xacro:property name="prop_mesh_file" value="file://$(find lolo_stonefish_sim)/data/lolo_auv/mesh/propeller.obj"/>
-  <xacro:property name="fin_mesh_file" value="file://$(find lolo_stonefish_sim)/data/lolo_auv/mesh/fin.obj"/>
-  <xacro:property name="back_fin_mesh_file" value="file://$(find lolo_stonefish_sim)/data/lolo_auv/mesh/back_fin.obj"/>
+  <xacro:property name="visual_mesh_file" value="file://$(find lolo_description)/mesh/lolo_hull.dae"/>
+  <xacro:property name="prop_port_mesh_file" value="file://$(find lolo_description)/mesh/lolo_port_propeller.dae"/>
+  <xacro:property name="prop_strb_mesh_file" value="file://$(find lolo_description)/mesh/lolo_strb_propeller.dae"/>
+  <xacro:property name="rudder_mesh_file" value="file://$(find lolo_description)/mesh/lolo_rudder.dae"/>
+  <xacro:property name="elevon_port_mesh_file" value="file://$(find lolo_description)/mesh/lolo_port_elevon.dae"/>
+  <xacro:property name="elevon_strb_mesh_file" value="file://$(find lolo_description)/mesh/lolo_strb_elevon.dae"/>
+  <xacro:property name="elevator_mesh_file" value="file://$(find lolo_description)/mesh/lolo_elevator.dae"/>
   <link name="$(arg robot_namespace)/base_link">
     <visual>
@@ -15,15 +18,18 @@
   <link name="$(arg robot_namespace)/dvl_link"/>
   <link name="$(arg robot_namespace)/compass_link"/>
-  <!--<link name="$(arg robot_namespace)/fls_link"/>-->
+  <link name="$(arg robot_namespace)/fls_link"/>
   <link name="$(arg robot_namespace)/imu_link"/>
   <link name="$(arg robot_namespace)/pressure_link"/>
   <link name="$(arg robot_namespace)/gps_link"/>
+  <link name="$(arg robot_namespace)/mbes_link"/>
+  <link name="$(arg robot_namespace)/usbl_link"/>
+  <!--For docking experiments.-->
   <link name="$(arg robot_namespace)/camera_link"/>
+  <!--End For docking experiments.-->
   <link name="$(arg robot_namespace)/elevator">
     <visual>
-      <origin xyz="0 0 0" rpy="${0.5*pi} 0 0" />
-      <!--<origin rpy="-1.5707 0.0 0.0" xyz="-2.68 0.0 0.0"/>-->
+      <origin xyz="0 0 0" rpy="0 0 0" />
       <geometry>
-        <mesh filename="${back_fin_mesh_file}" scale="1 1 1"/>
+        <mesh filename="${elevator_mesh_file}" scale="1 1 1"/>
       </geometry>
     </visual>
@@ -31,8 +37,7 @@
   <link name="$(arg robot_namespace)/rudder_stbd">
     <visual>
-      <origin xyz="0 0 0" rpy="${0.5*pi} 0 0" />
-      <!--<origin rpy="0.0 0.0 0.0" xyz="-2.4 -0.275 0.0"/>-->
+      <origin xyz="0 0 0" rpy="0 0 0" />
       <geometry>
-        <mesh filename="${fin_mesh_file}" scale="1 1 1"/>
+        <mesh filename="${rudder_mesh_file}" scale="1 1 1"/>
       </geometry>
     </visual>
@@ -40,35 +45,15 @@
   <link name="$(arg robot_namespace)/rudder_port">
     <visual>
-      <!--<origin rpy="0.0 0.0 0.0" xyz="-2.4 0.275 0.0"/>-->
-      <origin xyz="0 0 0" rpy="${0.5*pi} 0 0" />
+      <origin xyz="0 0 0" rpy="0 0 0" />
       <geometry>
-        <mesh filename="${fin_mesh_file}" scale="1 1 1"/>
+        <mesh filename="${rudder_mesh_file}" scale="1 1 1"/>
       </geometry>
     </visual>
   </link>
-  <!--
-  <link name="$(arg robot_namespace)/fin2">
-    <visual>
-      <origin xyz="0 0 0" rpy="${0.5*pi} 0 0" />
-      <geometry>
-        <mesh filename="${fin_mesh_file}" scale="1 1 1"/>
-      </geometry>
-    </visual>
-  </link>
-  <link name="$(arg robot_namespace)/fin3">
-    <visual>
-      <origin xyz="0 0 0" rpy="${0.5*pi} 0 0" />
-      <geometry>
-        <mesh filename="${fin_mesh_file}" scale="1 1 1"/>
-      </geometry>
-    </visual>
-  </link>
-  -->
   <link name="$(arg robot_namespace)/elevon_stbd">
     <visual>
-      <origin xyz="0 0 0" rpy="${0.5*pi} 0 0" />
-      <!--<origin rpy="1.5707 0.0 0.0" xyz="-0.8 -0.5 0.0"/>-->
+      <origin xyz="0 0 0" rpy="0 0 0" />
       <geometry>
-        <mesh filename="${fin_mesh_file}" scale="1 1 1"/>
+        <mesh filename="${elevon_strb_mesh_file}" scale="1 1 1"/>
       </geometry>
     </visual>
@@ -76,8 +61,7 @@
   <link name="$(arg robot_namespace)/elevon_port">
     <visual>
-      <origin xyz="0 0 0" rpy="${0.5*pi} 0 0" />
-      <!--<origin rpy="-1.5707 0.0 0.0" xyz="-0.8 0.5 0.0"/>-->
+      <origin xyz="0 0 0" rpy="0 0 0" />
       <geometry>
-        <mesh filename="${fin_mesh_file}" scale="1 1 1"/>
+        <mesh filename="${elevon_port_mesh_file}" scale="1 1 1"/>
       </geometry>
     </visual>
@@ -85,8 +69,7 @@
   <link name="$(arg robot_namespace)/thruster_port">
     <visual>
-      <origin xyz="0.0 0 0" rpy="0 0 ${pi}" />
-      <!--<origin rpy="0.0 0.0 3.1416" xyz="-2.85 0.275 0.0"/>-->
+      <origin xyz="0.0 0 0" rpy="0 0 0" />
       <geometry>
-        <mesh filename="${prop_mesh_file}" scale="1 1 1"/>
+        <mesh filename="${prop_port_mesh_file}" scale="1 1 1"/>
       </geometry>
     </visual>
@@ -94,8 +77,7 @@
   <link name="$(arg robot_namespace)/thruster_stbd">
     <visual>
-      <origin xyz="0.0 0 0" rpy="0 0 ${pi}" />
-      <!--<origin rpy="0.0 0.0 3.1416" xyz="-2.85 -0.275 0.0"/>-->
+      <origin xyz="0.0 0 0" rpy="0 0 0" />
       <geometry>
-        <mesh filename="${prop_mesh_file}" scale="1 1 1"/>
+        <mesh filename="${prop_strb_mesh_file}" scale="1 1 1"/>
       </geometry>
     </visual>
@@ -103,19 +85,19 @@
   <!-- Mount a 3D pose sensor -->
   <link name="$(arg robot_namespace)/pose_sensor_link">
-    <!--<visual>-->
-      <!--<geometry>-->
-        <!--<box size="0.01 0.01 0.01" />-->
-      <!--</geometry>-->
-    <!--</visual>-->
+    <visual>
+      <geometry>
+        <box size="0.01 0.01 0.01" />
+      </geometry>
+    </visual>
   </link>
   <joint name="$(arg robot_namespace)/elevator_joint" type="revolute">
-    <origin xyz="-2.68 0.0 0.0" rpy="${0.5*pi} 0 0" />
+    <origin xyz="-0.6476 0.0 0.0135" rpy="0 0 0" />
     <parent link="$(arg robot_namespace)/base_link" />
     <child link="$(arg robot_namespace)/elevator" />
     <limit effort="0" lower="-${pi/4.0}" upper="${pi/4.0}" velocity="0"/>
-    <axis xyz="0 0 1"/>
+    <axis xyz="0 1 0"/>
   </joint>
   <joint name="$(arg robot_namespace)/rudder_stbd_joint" type="revolute">
-    <origin xyz="-2.4 -0.275 0.0" rpy="0 0 0" />
+    <origin xyz="-0.3278 -0.253 0.129" rpy="0 0 0" />
     <parent link="$(arg robot_namespace)/base_link" />
     <child link="$(arg robot_namespace)/rudder_stbd" />
@@ -124,5 +106,5 @@
   </joint>
   <joint name="$(arg robot_namespace)/rudder_port_joint" type="revolute">
-    <origin xyz="-2.4 0.275 0.0" rpy="0 0 0" />
+    <origin xyz="-0.3278 0.253 0.129" rpy="0 0 0" />
     <parent link="$(arg robot_namespace)/base_link" />
     <child link="$(arg robot_namespace)/rudder_port" />
@@ -130,37 +112,21 @@
     <axis xyz="0 0 1"/>
   </joint>
-  <!--
-  <joint name="$(arg robot_namespace)/fin2_joint" type="revolute">
-    <origin xyz="-2.4 -0.275 -0.034" rpy="${pi} 0 0" />
-    <parent link="$(arg robot_namespace)/base_link" />
-    <child link="$(arg robot_namespace)/fin2" />
-    <limit effort="0" lower="-${pi/4.0}" upper="${pi/4.0}" velocity="0"/>
-    <axis xyz="0 0 1"/>
-  </joint>
-  <joint name="$(arg robot_namespace)/fin3_joint" type="revolute">
-    <origin xyz="-2.4 0.275 0.0" rpy="${pi} 0 0" />
-    <parent link="$(arg robot_namespace)/base_link" />
-    <child link="$(arg robot_namespace)/fin3" />
-    <limit effort="0" lower="-${pi/4.0}" upper="${pi/4.0}" velocity="0"/>
-    <axis xyz="0 0 1"/>
-  </joint>
-  -->
   <joint name="$(arg robot_namespace)/elevon_stbd_joint" type="revolute">
-    <origin xyz="-0.8 -0.5 0.0" rpy="${0.5*pi} 0 0" />
+    <origin xyz="-0.3733 -0.4035 0.01349" rpy="0 0 -0.19652" />
     <parent link="$(arg robot_namespace)/base_link" />
     <child link="$(arg robot_namespace)/elevon_stbd" />
     <limit effort="0" lower="-${pi/4.0}" upper="${pi/4.0}" velocity="0"/>
-    <axis xyz="0 0 1"/>
+    <axis xyz="0 1 0"/>
   </joint>
   <joint name="$(arg robot_namespace)/elevon_port_joint" type="revolute">
-    <origin xyz="-0.8 0.5 0.0" rpy="${-0.5*pi} 0 0" />
+    <origin xyz="-0.3733 0.4035 0.01349" rpy="0 0 0.19652" />
     <parent link="$(arg robot_namespace)/base_link" />
     <child link="$(arg robot_namespace)/elevon_port" />
     <limit effort="0" lower="-${pi/4.0}" upper="${pi/4.0}" velocity="0"/>
-    <axis xyz="0 0 1"/>
+    <axis xyz="0 1 0"/>
   </joint>
   <!-- Propeller -->
   <joint name="$(arg robot_namespace)/thruster_stbd_joint" type="continuous">
-    <origin xyz="-2.85 -0.275 0" rpy="0 0 0" />
+    <origin xyz="-0.9056 -0.2754 0.013678" rpy="0 0 0" />
     <axis xyz="1 0 0"/>
     <parent link="$(arg robot_namespace)/base_link"/>
@@ -168,5 +134,5 @@
   </joint>
   <joint name="$(arg robot_namespace)/thruster_port_joint" type="continuous">
-    <origin xyz="-2.85 0.275 0" rpy="0 0 0" />
+    <origin xyz="-0.9056 0.2754 0.013678" rpy="0 0 0" />
     <axis xyz="1 0 0"/>
     <parent link="$(arg robot_namespace)/base_link"/>
@@ -180,5 +146,5 @@
   </joint>
   <joint name="$(arg robot_namespace)/dvl_joint" type="fixed">
-    <origin rpy="0.0 0.0 0.0" xyz="1.25 0.0 -0.07"/>
+    <origin xyz="0.805 -0.025 -0.245" rpy="3.14159 0 0" />
     <parent link="$(arg robot_namespace)/base_link"/>
     <child link="$(arg robot_namespace)/dvl_link"/>
@@ -189,28 +155,40 @@
     <child link="$(arg robot_namespace)/compass_link"/>
   </joint>
-  <!--<joint name="$(arg robot_namespace)/fls_joint" type="fixed">-->
-    <!--<origin xyz="0 0 0" rpy="0 0 0" />-->
-    <!--<parent link="$(arg robot_namespace)/base_link"/>-->
-    <!--<child link="$(arg robot_namespace)/fls_link"/>-->
-  <!--</joint>-->
+  <joint name="$(arg robot_namespace)/fls_joint" type="fixed">
+    <origin xyz="0 0 0" rpy="0 0 0" />
+    <parent link="$(arg robot_namespace)/base_link"/>
+    <child link="$(arg robot_namespace)/fls_link"/>
+  </joint>
   <joint name="$(arg robot_namespace)/imu_joint" type="fixed">
-    <origin rpy="0.0 0.0 0.0" xyz="0.9 0.0 0.0"/>
+    <origin xyz="0 0 0" rpy="3.14159 0 0" />
     <parent link="$(arg robot_namespace)/base_link"/>
     <child link="$(arg robot_namespace)/imu_link"/>
   </joint>
   <joint name="$(arg robot_namespace)/pressure_joint" type="fixed">
-    <origin rpy="0.0 0.0 0.0" xyz="0.3 0.0 0.07"/>
+    <origin xyz="0 0 0" rpy="0 0 0" />
     <parent link="$(arg robot_namespace)/base_link"/>
     <child link="$(arg robot_namespace)/pressure_link"/>
   </joint>
   <joint name="$(arg robot_namespace)/gps_joint" type="fixed">
-    <origin rpy="0.0 0.0 0.0" xyz="1.2 0.0 0.08"/>
+    <origin xyz="0.836 0 0.44" rpy="0 0 0" />
     <parent link="$(arg robot_namespace)/base_link"/>
     <child link="$(arg robot_namespace)/gps_link"/>
   </joint>
+  <joint name="$(arg robot_namespace)/mbes_joint" type="fixed">
+    <origin xyz="2.523 0.0155 -0.302" rpy="3.14159 1.53589 0" />
+    <parent link="$(arg robot_namespace)/base_link"/>
+    <child link="$(arg robot_namespace)/mbes_link"/>
+  </joint>
+  <joint name="$(arg robot_namespace)/usbl_joint" type="fixed">
+    <origin xyz="0.389 0.002 0.337" rpy="0 0 0" />
+    <parent link="$(arg robot_namespace)/base_link"/>
+    <child link="$(arg robot_namespace)/usbl_link"/>
+  </joint>
+  <!--For docking experiments.-->
   <joint name="$(arg robot_namespace)/camera_joint" type="fixed">
-    <origin rpy="-1.5707 0.0 1.5707" xyz="-2.5 0.0 0.33"/>
+    <origin rpy="-1.5707 0.0 1.5707" xyz="0.0 0.0 0.33"/>
     <parent link="$(arg robot_namespace)/base_link"/>
     <child link="$(arg robot_namespace)/camera_link"/>
   </joint>
+  <!--End for docking experiments.-->
 </robot>

File: sam_stonefish_sim/data/sam_auv/sam_auv.urdf.xacro (robot description, xacro)
@@ -1,100 +1,60 @@
 <?xml version="1.0"?>
 <robot name="sam_auv" xmlns:xacro="http://www.ros.org/wiki/xacro">
-  <!-- ECA 5E Micro mnipulator -->
-  <!-- links -->
-  <xacro:property name="visual_mesh_file" value="file://$(find sam_stonefish_sim)/data/sam_auv/mesh/sam_body.obj"/>
+  <!-- Meshes. -->
+  <xacro:property name="visual_mesh_file" value="file://$(find sam_description)/mesh/SAM_HULL.dae"/>
+  <xacro:property name="prop_nozzle" value="file://$(find sam_description)/mesh/SAM_NOZZLE.dae"/>
+  <xacro:property name="front_prop" value="file://$(find sam_description)/mesh/SAM_FRONTPROP.dae"/>
+  <xacro:property name="back_prop" value="file://$(find sam_description)/mesh/SAM_BACKPROP.dae"/>
+  <!-- Links. -->
   <link name="$(arg robot_namespace)/base_link">
     <visual>
-      <origin rpy="0.0 0.0 0.0" xyz="0.0 0.0 0.0"/>
+      <origin xyz="0 0 0" rpy="0 0 0"/>
       <geometry>
-        <mesh filename="${visual_mesh_file}" scale="1 1 1" />
+        <mesh filename="${visual_mesh_file}" scale="1 1 1"/>
       </geometry>
     </visual>
   </link>
-  <link name="$(arg robot_namespace)/thruster_yaw_link">
+  <link name="$(arg robot_namespace)/thruster_link">
+    <visual>
+      <origin xyz="0 0 0" rpy="0 0 0"/>
+      <geometry>
+        <mesh filename="${prop_nozzle}" scale="1 1 1"/>
+      </geometry>
+    </visual>
   </link>
-  <link name="$(arg robot_namespace)/thruster_link">
+  <link name="$(arg robot_namespace)/front_prop_link">
+    <visual>
+      <origin xyz="0 0 0" rpy="0 0 0"/>
+      <geometry>
+        <mesh filename="${front_prop}" scale="1 1 1"/>
+      </geometry>
+    </visual>
   </link>
-  <link name="$(arg robot_namespace)/battery_link">
+  <link name="$(arg robot_namespace)/back_prop_link">
+    <visual>
+      <origin xyz="0 0 0" rpy="0 0 0"/>
+      <geometry>
+        <mesh filename="${back_prop}" scale="1 1 1"/>
+      </geometry>
+    </visual>
   </link>
-  <link name="$(arg robot_namespace)/tcg1_link">
-  </link>
-  <link name="$(arg robot_namespace)/tcg2_link">
-  </link>
-  <link name="$(arg robot_namespace)/multibeam_down_link">
-  </link>
-  <link name="$(arg robot_namespace)/pressure_link">
-  </link>
-  <link name="$(arg robot_namespace)/dvl_link">
-  </link>
-  <link name="$(arg robot_namespace)/imu_link">
-  </link>
-  <link name="$(arg robot_namespace)/sbg_link">
-  </link>
-<!--   <link name="$(arg robot_namespace)/mag_link">
-  </link> -->
-  <link name="$(arg robot_namespace)/gps_link">
-  </link>
-  <link name="$(arg robot_namespace)/camera_down_link">
-  </link>
-  <link name="$(arg robot_namespace)/camera_front_right_link">
-  </link>
-  <link name="$(arg robot_namespace)/camera_front_left_link">
-  </link>
-  <link name="$(arg robot_namespace)/docking_station_link">
-  </link>
-  <link name="$(arg robot_namespace)/usbl_link">
-  </link>
-  <joint name="$(arg robot_namespace)/multibeam_down_joint" type="fixed">
-    <parent link="$(arg robot_namespace)/base_link"/>
-    <child link="$(arg robot_namespace)/multibeam_down_link"/>
-    <origin rpy="0.0 1.5707 0.0" xyz="1.20 0.0 -0.07"/>
-  </joint>
-  <joint name="$(arg robot_namespace)/pressure_joint" type="fixed">
-    <parent link="$(arg robot_namespace)/base_link"/>
-    <child link="$(arg robot_namespace)/pressure_link"/>
-    <origin rpy="0.0 0.0 0.0" xyz="0.3 0.0 0.07"/>
-  </joint>
-  <joint name="$(arg robot_namespace)/dvl_joint" type="fixed">
-    <parent link="$(arg robot_namespace)/base_link"/>
-    <child link="$(arg robot_namespace)/dvl_link"/>
-    <origin rpy="0.0 0.0 0.0" xyz="1.25 0.0 -0.07"/>
-  </joint>
-  <joint name="$(arg robot_namespace)/imu_joint" type="fixed">
-    <parent link="$(arg robot_namespace)/base_link"/>
-    <child link="$(arg robot_namespace)/imu_link"/>
-    <origin rpy="0.0 0.0 0.0" xyz="0.9 0.0 0.0"/>
-  </joint>
-  <joint name="$(arg robot_namespace)/sbg_joint" type="fixed">
-    <parent link="$(arg robot_namespace)/base_link"/>
-    <child link="$(arg robot_namespace)/sbg_link"/>
-    <origin rpy="0.0 0.0 0.0" xyz="0.472 0 0.03"/>
-  </joint>
-    <!-- Compass doesn't seem to have a ROS parser -->
-<!--   <joint name="$(arg robot_namespace)/mag_joint" type="fixed">
-    <parent link="$(arg robot_namespace)/base_link"/>
-    <child link="$(arg robot_namespace)/mag_link"/>
-    <origin rpy="0.0 0.0 0.0" xyz="0.472 0 0.03"/>
-  </joint> -->
-  <joint name="$(arg robot_namespace)/gps_joint" type="fixed">
-    <parent link="$(arg robot_namespace)/base_link"/>
-    <child link="$(arg robot_namespace)/gps_link"/>
-    <origin rpy="0.0 1.5707 0.0" xyz="1.2 0.0 0.08"/>
-  </joint>
-  <joint name="$(arg robot_namespace)/camera_down_joint" type="fixed">
-    <parent link="$(arg robot_namespace)/base_link"/>
-    <child link="$(arg robot_namespace)/camera_down_link"/>
-    <origin rpy="3.1416 0.0 -1.5707" xyz="1.15 0.0 -0.07"/>
-  </joint>
-  <joint name="$(arg robot_namespace)/camera_front_right_joint" type="fixed">
-    <parent link="$(arg robot_namespace)/base_link"/>
-    <child link="$(arg robot_namespace)/camera_front_right_link"/>
-    <origin rpy="1.3 3.1416 2.3416" xyz="1.32 0.05 0.005"/>
-  </joint>
-  <joint name="$(arg robot_namespace)/camera_front_left_joint" type="fixed">
-    <parent link="$(arg robot_namespace)/base_link"/>
-    <child link="$(arg robot_namespace)/camera_front_left_link"/>
-    <origin rpy="1.3 3.1416 0.8" xyz="1.32 -0.05 0.005"/>
-  </joint>
+  <link name="$(arg robot_namespace)/thruster_yaw_link"/>
+  <link name="$(arg robot_namespace)/battery_link"/>
+  <link name="$(arg robot_namespace)/tcg1_link"/>
+  <link name="$(arg robot_namespace)/tcg2_link"/>
+  <link name="$(arg robot_namespace)/pressure_link"/>
+  <link name="$(arg robot_namespace)/dvl_link"/>
+  <link name="$(arg robot_namespace)/sidescan_link"/>
+  <link name="$(arg robot_namespace)/imu_link"/>
+  <link name="$(arg robot_namespace)/sbg_link"/>
+  <link name="$(arg robot_namespace)/gps_link"/>
+  <link name="$(arg robot_namespace)/uw_gps_link"/>
+  <link name="$(arg robot_namespace)/camera_down_link"/>
+  <link name="$(arg robot_namespace)/camera_front_right_link"/>
+  <link name="$(arg robot_namespace)/camera_front_left_link"/>
+  <!--Fod docking experiments.-->
+  <link name="$(arg robot_namespace)/docking_station_link"/>
+  <link name="$(arg robot_namespace)/usbl_link"/>
+  <!--End For docking experiments.-->
   <joint name="$(arg robot_namespace)/thruster_yaw_joint" type="revolute">
     <parent link="$(arg robot_namespace)/base_link"/>
@@ -111,4 +71,67 @@
     <limit lower="-0.2" upper="0.2" velocity="0.2" effort="1.0"/>
   </joint>
+  <joint name="$(arg robot_namespace)/front_prop_joint" type="continuous">
+    <parent link="$(arg robot_namespace)/base_link"/>
+    <child link="$(arg robot_namespace)/front_prop_link"/>
+    <origin rpy="0.0 0.0 0.0" xyz="-0.056 0 0"/>
+    <axis xyz="1 0 0"/>
+  </joint>
+  <joint name="$(arg robot_namespace)/back_prop_joint" type="continuous">
+    <parent link="$(arg robot_namespace)/base_link"/>
+    <child link="$(arg robot_namespace)/back_prop_link"/>
+    <origin rpy="0.0 0.0 0.0" xyz="-0.074 0 0"/>
+    <axis xyz="1 0 0"/>
+  </joint>
+  <joint name="$(arg robot_namespace)/pressure_joint" type="fixed">
+    <parent link="$(arg robot_namespace)/base_link"/>
+    <child link="$(arg robot_namespace)/pressure_link"/>
+    <origin rpy="0.0 0.0 0.0" xyz="0.174 0.025 0.057"/>
+  </joint>
+  <joint name="$(arg robot_namespace)/dvl_joint" type="fixed">
+    <parent link="$(arg robot_namespace)/base_link"/>
+    <child link="$(arg robot_namespace)/dvl_link"/>
+    <origin rpy="0.0 0.0 0.0" xyz="1.25 0.0 -0.063"/>
+  </joint>
+  <!--Sidescan acoustic center, i.e. intersection between both sidescan centers.-->
+  <joint name="$(arg robot_namespace)/sidescan_joint" type="fixed">
+    <parent link="$(arg robot_namespace)/base_link"/>
+    <child link="$(arg robot_namespace)/sidescan_link"/>
+    <origin rpy="0.0 0.0 0.0" xyz="0.634 0.0 0.0"/>
+  </joint>
+  <joint name="$(arg robot_namespace)/imu_joint" type="fixed">
+    <parent link="$(arg robot_namespace)/base_link"/>
+    <child link="$(arg robot_namespace)/imu_link"/>
+    <origin rpy="0.0 0.0 0.0" xyz="0.917 0.0 -0.036"/>
+  </joint>
+  <joint name="$(arg robot_namespace)/sbg_joint" type="fixed">
+    <parent link="$(arg robot_namespace)/base_link"/>
+    <child link="$(arg robot_namespace)/sbg_link"/>
+    <origin rpy="0.0 0.0 0.0" xyz="1.137 0.0 0.002"/>
+  </joint>
+  <joint name="$(arg robot_namespace)/gps_joint" type="fixed">
+    <parent link="$(arg robot_namespace)/base_link"/>
+    <child link="$(arg robot_namespace)/gps_link"/>
+    <origin rpy="0.0 0.0 0.0" xyz="1.205 0.0 0.071"/>
+  </joint>
+  <joint name="$(arg robot_namespace)/uw_gps_joint" type="fixed">
+    <parent link="$(arg robot_namespace)/base_link"/>
+    <child link="$(arg robot_namespace)/uw_gps_link"/>
+    <origin rpy="0.0 0.0 0.0" xyz="0.275 0.0 0.078"/>
+  </joint>
+  <joint name="$(arg robot_namespace)/camera_down_joint" type="fixed">
+    <parent link="$(arg robot_namespace)/base_link"/>
+    <child link="$(arg robot_namespace)/camera_down_link"/>
+    <origin rpy="3.1416 0.0 -1.5707" xyz="1.1385 0.0 -0.052"/>
+  </joint>
+  <joint name="$(arg robot_namespace)/camera_front_left_joint" type="fixed">
+    <parent link="$(arg robot_namespace)/base_link"/>
+    <child link="$(arg robot_namespace)/camera_front_left_link"/>
+    <origin rpy="1.3 3.1416 2.3416" xyz="1.313 0.048 -0.007"/>
+  </joint>
+  <joint name="$(arg robot_namespace)/camera_front_right_joint" type="fixed">
+    <parent link="$(arg robot_namespace)/base_link"/>
+    <child link="$(arg robot_namespace)/camera_front_right_link"/>
+    <origin rpy="1.3 3.1416 0.8" xyz="1.313 -0.048 -0.007"/>
+  </joint>
   <joint name="$(arg robot_namespace)/lcg_joint" type="prismatic">
     <parent link="$(arg robot_namespace)/base_link"/>
@@ -121,5 +144,5 @@
     <parent link="$(arg robot_namespace)/base_link"/>
     <child link="$(arg robot_namespace)/tcg1_link"/>
-    <origin rpy="0.0 0.0 0.0" xyz="0.48 0.0 0.0"/>
+    <origin rpy="0.0 0.0 0.0" xyz="0.582 0.0 0.0"/>
     <axis xyz="1 0 0"/>
     <limit lower="-1.6" upper="1.6" velocity="0.2" effort="1.0"/>
@@ -128,12 +151,13 @@
     <parent link="$(arg robot_namespace)/base_link"/>
     <child link="$(arg robot_namespace)/tcg2_link"/>
-    <origin rpy="0.0 0.0 0.0" xyz="0.46 0.0 0.0"/>
+    <origin rpy="0.0 0.0 0.0" xyz="0.552 0.0 0.0"/>
     <axis xyz="1 0 0"/>
     <limit lower="-1.6" upper="1.6" velocity="0.2" effort="1.0"/>
   </joint>
+  <!--Fod docking experiments.-->
   <joint name="$(arg robot_namespace)/docking_station_joint" type="fixed">
     <parent link="$(arg robot_namespace)/base_link"/>
     <child link="$(arg robot_namespace)/docking_station_link"/>
-    <origin rpy="-1.5708 0 1.5708" xyz="-0.045 -0.0025 0.0"/>
+    <origin rpy="-1.5708 0 1.5708" xyz="1.0 0.0 0.0"/>
   </joint>
   <joint name="$(arg robot_namespace)/usbl_joint" type="fixed">
@@ -142,3 +166,4 @@
     <origin rpy="0 0 0" xyz="0 0 0"/>
   </joint>
+  <!--End For docking experiments.-->
 </robot>
