Commit message: Update XML and URDF to include docking link and camera link

File: lolo_stonefish_sim/data/lolo_auv/lolo_auv.urdf.xacro (robot description, xacro)
@@ -26,4 +26,5 @@
   <!--For docking experiments.-->
   <link name="$(arg robot_namespace)/camera_link"/>
+  <link name="$(arg robot_namespace)/docking_link"/>
   <!--End For docking experiments.-->
   <link name="$(arg robot_namespace)/elevator">
@@ -191,4 +192,9 @@
     <child link="$(arg robot_namespace)/camera_link"/>
   </joint>
+  <joint name="$(arg robot_namespace)/docking_joint" type="fixed">
+    <origin rpy="-1.5707 0.0 1.5707" xyz="2.5 0.0 0.0"/>
+    <parent link="$(arg robot_namespace)/base_link"/>
+    <child link="$(arg robot_namespace)/docking_link"/>
+  </joint>
   <!--End for docking experiments.-->
 </robot>
