Commit message: Preparing for simulations on VM

File: sam_stonefish_sim/data/sam_auv/sam_auv.urdf.xacro (robot description, xacro)
@@ -43,4 +43,6 @@
   </link>
   <link name="$(arg robot_namespace)/docking_station_link">
+  </link>
+  <link name="$(arg robot_namespace)/usbl_link">
   </link>
   <joint name="$(arg robot_namespace)/multibeam_down_joint" type="fixed">
@@ -135,3 +137,8 @@
     <origin rpy="-1.5708 0 1.5708" xyz="-0.045 -0.0025 0.0"/>
   </joint>
+  <joint name="$(arg robot_namespace)/usbl_joint" type="fixed">
+    <parent link="$(arg robot_namespace)/base_link"/>
+    <child link="$(arg robot_namespace)/usbl_link"/>
+    <origin rpy="0 0 0" xyz="0 0 0"/>
+  </joint>
 </robot>

Commit message: Update XML and URDF to include docking link and camera link

File: sam_stonefish_sim/data/sam_auv/sam_auv.urdf.xacro (robot description, xacro)
@@ -54,6 +54,6 @@
   <link name="$(arg robot_namespace)/camera_front_left_link"/>
   <!--Fod docking experiments.-->
-  <link name="$(arg robot_namespace)/docking_station_link"/>
   <link name="$(arg robot_namespace)/usbl_link"/>
+  <link name="$(arg robot_namespace)/camera_link"/>
   <!--End For docking experiments.-->
   <joint name="$(arg robot_namespace)/thruster_yaw_joint" type="revolute">
@@ -156,9 +156,4 @@
   </joint>
   <!--Fod docking experiments.-->
-  <joint name="$(arg robot_namespace)/docking_station_joint" type="fixed">
-    <parent link="$(arg robot_namespace)/base_link"/>
-    <child link="$(arg robot_namespace)/docking_station_link"/>
-    <origin rpy="-1.5708 0 1.5708" xyz="1.0 0.0 0.0"/>
-  </joint>
   <joint name="$(arg robot_namespace)/usbl_joint" type="fixed">
     <parent link="$(arg robot_namespace)/base_link"/>
@@ -166,4 +161,9 @@
     <origin rpy="0 0 0" xyz="0 0 0"/>
   </joint>
+  <joint name="$(arg robot_namespace)/camera_joint" type="fixed">
+    <parent link="$(arg robot_namespace)/base_link"/>
+    <child link="$(arg robot_namespace)/camera_link"/>
+    <origin rpy="-1.5707 0 1.5707" xyz="0 0 0.10"/>
+  </joint>
   <!--End For docking experiments.-->
 </robot>

Commit message: Update params to fit static docking scenario

File: sam_stonefish_sim/data/sam_auv/sam_auv.urdf.xacro (robot description, xacro)
@@ -53,7 +53,8 @@
   <link name="$(arg robot_namespace)/camera_front_right_link"/>
   <link name="$(arg robot_namespace)/camera_front_left_link"/>
-  <!--Fod docking experiments.-->
+  <!--For docking experiments.-->
   <link name="$(arg robot_namespace)/usbl_link"/>
   <link name="$(arg robot_namespace)/camera_link"/>
+  <link name="$(arg robot_namespace)/camera_front_link"/>
   <!--End For docking experiments.-->
   <joint name="$(arg robot_namespace)/thruster_yaw_joint" type="revolute">
@@ -134,4 +135,9 @@
     <origin rpy="1.3 3.1416 0.8" xyz="1.313 -0.048 -0.007"/>
   </joint>
+  <joint name="$(arg robot_namespace)/camera_front_joint" type="fixed">
+    <parent link="$(arg robot_namespace)/base_link"/>
+    <child link="$(arg robot_namespace)/camera_front_link"/>
+    <origin rpy="-1.5707 0.0 -1.5707" xyz="1.313 0.0 0.0"/>
+  </joint>
   <joint name="$(arg robot_namespace)/lcg_joint" type="prismatic">
     <parent link="$(arg robot_namespace)/base_link"/>
